Commit message: Feat: Meta Quest teleop control implementation
Build reduced URDF to account for lower DOF on so101

Fix: Cleanup URDF setup and usage to account for 5DOF so101

Update params for teleop

Added EEF link to URDF

Feat: viser tool to check teleop control in simulation

Feat: added config params for dual-arm setup

Feat: dual-arm variants of utils

Feat: update IK solver to account for dual-arm setup

Feat: dual-arm variants of utils

Feat: additional utils for quest integration

Feat: Update quest reader to account for dual-arm setup

Feat: teleop dual-arm so101 setup using both meta quest controllers

Feat: Use neuracore to collect data from dual-arm so101 setup

Fix: reset joint 4 costs to 0

Feat: update visualizer to support dual-arm setup

Feat: enable dual-arm visualization in Viser

Feat: Dual arm URDF + meshes

Fix: enable camera and cleanup code

fix: corrected orientations for quest controls for dual arm setup

Fix: Updated readme with instructions for new examples

Fix: Removed meta_quest_teleop repo local copy

fix: added meta quest teleop repo to env yaml

File: so101_description/robot.urdf (robot description, URDF)
Before this commit: robot so101_new_calib, 8 links, 7 joints
Links:
- added link eef_link, mass 1e-9
Joints:
- added joint eef_joint: type fixed, parent gripper_frame_link, child eef_link, origin xyz=0 0 0 rpy=-1.57 -1.57 0, axis 0 0 0
